File: cardEmulator.kicad_pcb (KiCad board)
At the start: 2 copper layers, 11.7 x 25.9 mm, 29 parts, among them J1 USB_B_Micro, SW1 SW_Push, U1 TPS613222A, U2 MCP73831-2-OT, U3 ATtiny85-20SU, U4 TPS3839DBZ, U5 DRV8835

Commit message: rev2 released
 - Fixed 5V boost converter footprint (U1, TPS5613222A) to be DBZ version, which is SOT23-5
 - Added better silkscreen documentation
Parts:
- C2: value C_Small -> 120pF
- C4: value C -> 10uF
- D4: value D_Schottky -> SMD22WS-TP
- R1: value CH_I_SET -> 47k
- R2: value R_US -> 5.1
- SW1: footprint custom3d:SW_SPST_PTS645 -> custom3d:SW_SPST_PTS645-custom-silkscreen
- U1: footprint Package_TO_SOT_SMD:SOT-23 -> Package_TO_SOT_SMD:SOT-23-5
- moved U1 0.53 mm to (117.7, 102.3), turned to 270 degrees
Connections:
- U1 pad 1: +5V -> Net-(D4-Pad2)
- U1 pad 2: Net-(D4-Pad2) -> GND
- U1 pad 3: GND -> (no net)
Other:
- board text added: "19.211"
- board text added: "github.co m/willemcvu/ magspoofmini"
- board text added: "rev2"
- board text removed: "Desg s"
- board text removed: "No"
- board text removed: "Refc."
- board text removed: "Space,no"
- board text removed: "WTech"
