File: cardEmulator.sch (KiCad schematic (older format))
At the start: 28 parts, among them J1 USB_B_Micro, SW1 SW_Push, U1 TPS613222A, U2 MCP73831-2-OT, U3 ATtiny85-20SU, U4 TPS3839DBZ, U5 DRV8835

Commit message: rev2 released
 - Fixed 5V boost converter footprint (U1, TPS5613222A) to be DBZ version, which is SOT23-5
 - Added better silkscreen documentation
Parts:
- U1: footprint Package_TO_SOT_SMD:SOT-23 -> Package_TO_SOT_SMD:SOT-23-5; symbol cardEmulator-rescue:TPS613222A-CUSTOM_IC -> cardEmulator-rescue:TPS613222A-DBV
Connections:
- net +5V: now also U1.4 (VOUT); no longer U1.1 (VOUT)
- net GND: now also U1.2 (GND); no longer U1.3 (GND)
- net at D4.2 (A), L1.2, R2.2: now also U1.1 (SW); no longer U1.2 (SW)
Changed lines of the file:
@@
 EESchema Schematic File Version 4
 LIBS:cardEmulator-cache
-EELAYER 26 0
+EELAYER 29 0
 EELAYER END
 $Descr A4 11693 8268
@@
 $EndComp
 $Comp
-L cardEmulator-rescue:TPS613222A-CUSTOM_IC U1
+L cardEmulator-rescue:TPS613222A-DBV U1
 U 1 1 5BCCC336
 P 2700 4300
 F 0 "U1" H 2700 4625 50  0000 C CNN
 F 1 "TPS613222A" H 2700 4534 50  0000 C CNN
-F 2 "Package_TO_SOT_SMD:SOT-23" H 2700 4300 50  0001 C CNN
+F 2 "Package_TO_SOT_SMD:SOT-23-5" H 2700 4300 50  0001 C CNN
 F 3 "" H 2700 4300 50  0001 C CNN
 	1    2700 4300
