File: kicad-board/v2.kicad_pcb (KiCad board)
At the start: 2 copper layers, 16.5 x 28.4 mm, 27 parts, among them J1 USB_B_Micro, J2 LiPO, Q1 Q_NMOS_GDS, SW1 SW_Push, U1 MCP73831-2-OT, U2 ATtiny85-20SU, U3 TPS6102x

Commit message: Made new board
Parts:
- R2: value R1 -> 1M
- R3: value R2 -> 180k
- R4: value R3 -> 1.6M
- R5: value R4 -> 180k
Connections:
- R5 pad 2: /BATT_LOW_LED -> GND

Commit message: Updated silkscreen, shipped board
Other:
- board text added: "rev2.1 19.224 W. Hillier"
- board text removed: "rev2 19.212 W. Hillier"
Changed lines of the file:
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@@
   )
   (setup
-    (last_trace_width 0.2032)
+    (last_trace_width 0.1524)
     (user_trace_width 0.2032)
     (user_trace_width 0.254)
@@
     (effects (font (size 1.651 1.651) (thickness 0.2286)) (justify mirror))
   )
-  (gr_text "rev2 19.212\nW. Hillier" (at 135.763 -46.736 270) (layer B.SilkS)
+  (gr_text "rev2.1 19.224\nW. Hillier" (at 135.763 -46.736 270) (layer B.SilkS)
     (effects (font (size 1.016 1.016) (thickness 0.1778)) (justify mirror))
   )
