File: kicad-board/v2_panelized.kicad_pcb (KiCad board)
At the start: 2 copper layers, 99.4 x 85.5 mm, 486 parts, among them J1 USB_B_Micro, J2 LiPO, Q1 Q_NMOS_GDS, SW1 SW_Push, U1 MCP73831-2-OT, U2 ATtiny85-20SU, U3 TPS6102x

Commit message: Updated silkscreen, shipped board
Parts:
- removed the D3 at (168.3, -18.1)
- removed the D3 at (201.4, -18.1)
- removed the R6 at (231.8, -1.22)
- removed the SW1 at (171.8, -10.6)
- added C6: 100u, Capacitor_SMD:C_1206_3216Metric, F.Cu at (197.1, -7.06)
- added Q1: Q_NMOS_GDS, Package_TO_SOT_SMD:SOT-23, F.Cu at (162.2, -39.2)
- added Q1: Q_NMOS_GDS, Package_TO_SOT_SMD:SOT-23, F.Cu at (228.5, -10.7)
- added U1: MCP73831-2-OT, Package_TO_SOT_SMD:SOT-23-5, F.Cu at (180.8, -22.9)
- D3: renamed from L1; value 6.8uH -> RED_LED; footprint footprints:L_B82462G4_6.3mmx3mm -> LED_SMD:LED_0603_1608Metric
- D3: renamed from Q1; value Q_NMOS_GDS -> RED_LED; footprint Package_TO_SOT_SMD:SOT-23 -> LED_SMD:LED_0603_1608Metric
- L1: renamed from Q1; value Q_NMOS_GDS -> 6.8uH; footprint Package_TO_SOT_SMD:SOT-23 -> footprints:L_B82462G4_6.3mmx3mm
- R6: renamed from RN1; value 1k -> R5; footprint Resistor_SMD:R_Cat16-4 -> Resistor_SMD:R_0603_1608Metric
- RN1: renamed from TP3; value COIL1 -> 1k; footprint TestPoint:TestPoint_Pad_3.0x3.0mm -> Resistor_SMD:R_Cat16-4; moved to F.Cu
- SW1: renamed from C6; value 100u -> SW_Push; footprint Capacitor_SMD:C_1206_3216Metric -> custom3d:SW_SPST_PTS645
- TP3: renamed from U1; value MCP73831-2-OT -> COIL1; footprint Package_TO_SOT_SMD:SOT-23-5 -> TestPoint:TestPoint_Pad_3.0x3.0mm; moved to B.Cu
- moved R6 76.2 mm to (231.8, -1.22), turned to 90 degrees
- moved D3 56.5 mm to (168.3, -18.1), turned to 180 degrees
- moved L1 53.6 mm to (188.4, 24.9), turned to 270 degrees
- moved D3 44.5 mm to (201.4, -18.1), turned to 180 degrees
- moved RN1 44.4 mm to (171.2, -47.4), turned to 180 degrees
- moved TP3 33.2 mm to (212.8, -31.9), turned to 270 degrees
- moved SW1 25.6 mm to (171.8, -10.6)
- moved L1 16.6 mm to (204.9, 24.9)
Connections:
- D3 pad 1: +VSW -> Net-(D3-Pad1)
- D3 pad 2: Net-(L1-Pad2) -> +5V
- D3 pad 1: Net-(Q1-Pad1) -> Net-(D3-Pad1)
- D3 pad 2: GND -> +5V
- L1 pad 1: Net-(Q1-Pad1) -> +VSW
- L1 pad 2: GND -> Net-(L1-Pad2)
- R6 pad 1: /CHG_LED -> +5V
- RN1 pad 1: +5V -> /CHG_LED
- SW1 pad 1: +5V -> +BATT
- SW1 pad 2: GND -> +VSW
- TP3 pad 1: /CHG_LED -> +5V
Other:
- board text added: "rev2.1 19.224 W. Hillier"
- board text removed: "rev2 19.212 W. Hillier"
