File: kicad-board/v2.sch (KiCad schematic (older format))
At the start: 27 parts, among them J1 USB_B_Micro, J2 LiPO, Q1 Q_NMOS_GDS, SW1 SW_Push, U1 MCP73831-2-OT, U2 ATtiny85-20SU, U3 TPS6102x

Commit message: Made new board
Parts:
- R2: value R1 -> 1M
- R3: value R2 -> 180k
- R4: value R3 -> 1.6M
- R5: value R4 -> 180k
- U2: symbol cardEmulator-rescue:ATtiny85-20SU-MCU_Microchip_ATtiny -> v2-rescue:ATtiny85-20SU-MCU_Microchip_ATtiny-cardEmulator-rescue
Connections:
- net BATT_LOW_LED: no longer R5.2
- net GND: now also R5.2
Changed lines of the file:
@@
 EESchema Schematic File Version 4
-LIBS:cardEmulator-cache
+LIBS:v2-cache
 EELAYER 29 0
 EELAYER END
@@
 $EndComp
 $Comp
-L cardEmulator-rescue:ATtiny85-20SU-MCU_Microchip_ATtiny U2
+L v2-rescue:ATtiny85-20SU-MCU_Microchip_ATtiny-cardEmulator-rescue U2
 U 1 1 5B86A5F1
 P 3800 1850
@@
 P 3100 4000
 F 0 "R2" H 3168 4046 50  0000 L CNN
-F 1 "R1" H 3168 3955 50  0000 L CNN
+F 1 "1M" H 3168 3955 50  0000 L CNN
 F 2 "Resistor_SMD:R_0603_1608Metric" V 3140 3990 50  0001 C CNN
 F 3 "~" H 3100 4000 50  0001 C CNN
@@
 P 3100 4300
 F 0 "R3" H 3168 4346 50  0000 L CNN
-F 1 "R2" H 3168 4255 50  0000 L CNN
+F 1 "180k" H 3168 4255 50  0000 L CNN
 F 2 "Resistor_SMD:R_0603_1608Metric" V 3140 4290 50  0001 C CNN
 F 3 "~" H 3100 4300 50  0001 C CNN
@@
 P 4650 4100
 F 0 "R5" H 4718 4146 50  0000 L CNN
-F 1 "R4" H 4718 4055 50  0000 L CNN
+F 1 "180k" H 4718 4055 50  0000 L CNN
 F 2 "Resistor_SMD:R_0603_1608Metric" V 4690 4090 50  0001 C CNN
 F 3 "~" H 4650 4100 50  0001 C CNN
@@
 P 4650 3800
 F 0 "R4" H 4718 3846 50  0000 L CNN
-F 1 "R3" H 4718 3755 50  0000 L CNN
+F 1 "1.6M" H 4718 3755 50  0000 L CNN
 F 2 "Resistor_SMD:R_0603_1608Metric" V 4690 3790 50  0001 C CNN
 F 3 "~" H 4650 3800 50  0001 C CNN
@@
 	5150 3650 5650 3650
 Connection ~ 5650 3650
-Wire Wire Line
-	4400 4250 4650 4250
-Connection ~ 4650 4250
 $Comp
 L Device:R_US R6
@@
 $EndComp
 Wire Wire Line
-	4650 4250 6050 4250
-Wire Wire Line
 	5650 3650 6050 3650
 Wire Wire Line
@@
 Wire Wire Line
 	6050 4100 6050 4250
-Connection ~ 6050 4250
 Wire Wire Line
 	6050 4250 6400 4250
@@
 Wire Wire Line
 	1350 4200 1350 4350
+$Comp
+L power:GND #PWR?
+U 1 1 5D5B800E
+P 4650 4250
+F 0 "#PWR?" H 4650 4000 50  0001 C CNN
+F 1 "GND" H 4655 4077 50  0000 C CNN
+F 2 "" H 4650 4250 50  0001 C CNN
+F 3 "" H 4650 4250 50  0001 C CNN
+	1    4650 4250
+	1    0    0    -1
+$EndComp
+Wire Wire Line
+	4400 4250 4500 4250
+Wire Wire Line
+	4500 4250 4500 4550
+Wire Wire Line
+	4500 4550 5500 4550
+Wire Wire Line
+	5500 4550 5500 4250
+Wire Wire Line
+	5500 4250 6050 4250
+Connection ~ 6050 4250
 $EndSCHEMATC

Commit message: Updated resistor values
Parts:
- R6: value R5 -> 1k
Changed lines of the file:
@@
 P 6050 3950
 F 0 "R6" H 6118 3996 50  0000 L CNN
-F 1 "R5" H 6118 3905 50  0000 L CNN
+F 1 "1k" H 6118 3905 50  0000 L CNN
 F 2 "Resistor_SMD:R_0603_1608Metric" V 6090 3940 50  0001 C CNN
 F 3 "~" H 6050 3950 50  0001 C CNN
@@
 	1350 4200 1350 4350
 $Comp
-L power:GND #PWR?
+L power:GND #PWR0106
 U 1 1 5D5B800E
 P 4650 4250
-F 0 "#PWR?" H 4650 4000 50  0001 C CNN
+F 0 "#PWR0106" H 4650 4000 50  0001 C CNN
 F 1 "GND" H 4655 4077 50  0000 C CNN
 F 2 "" H 4650 4250 50  0001 C CNN
